Commit message: libtaurob and the description package ported

File: taurob_tracker_description/urdf/tracker.urdf.xacro (robot description, xacro)
@@ -8,7 +8,7 @@
   <xacro:include filename="$(find taurob_tracker_description)/urdf/tracker_chassis.urdf.xacro"/>
   <xacro:include filename="$(find taurob_tracker_description)/urdf/tracker_arm.urdf.xacro"/>
-  <tracker_chassis_macro/>
-  <tracker_arm_macro parent="base_link">
+  <xacro:tracker_chassis_macro/>
+  <xacro:tracker_arm_macro parent="base_link">
     <origin xyz="0.12 0 0.185" rpy="0 0 ${M_PI/2}"/>
-  </tracker_arm_macro>
+  </xacro:tracker_arm_macro>
 </robot>

File: taurob_tracker_description/urdf/tracker_arm.urdf.xacro (robot description, xacro)
@@ -10,8 +10,4 @@
       <axis xyz="0 0 1"/>
       <limit lower="${-180 * M_PI / 180}" upper="${180 * M_PI / 180}" effort="1000" velocity="${1.0 * 110 * M_PI / 180}"/>
-      <!--        <safety_controller soft_lower_limit="${-168 * M_PI / 180}"
-				 soft_upper_limit="${168 * M_PI / 180}"
-				 k_position="${100}"
-				 k_velocity="${2}"/>-->
       <parent link="${parent}"/>
       <child link="arm_link_0"/>
@@ -38,8 +34,4 @@
       <axis xyz="1 0 0"/>
       <limit lower="${0 * M_PI / 180}" upper="${180 * M_PI / 180}" effort="1000" velocity="${1.0 * 110 * M_PI / 180}"/>
-      <!--        <safety_controller soft_lower_limit="${-168 * M_PI / 180}"
-				 soft_upper_limit="${168 * M_PI / 180}"
-				 k_position="${100}"
-				 k_velocity="${2}"/>-->
       <parent link="arm_link_0"/>
       <child link="arm_link_1"/>
@@ -66,8 +58,4 @@
       <axis xyz="-1 0 0"/>
       <limit lower="${0}" upper="${2 * M_PI}" effort="1000" velocity="${1.0 * 110 * M_PI / 180}"/>
-      <!--        <safety_controller soft_lower_limit="${-168 * M_PI / 180}"
-				 soft_upper_limit="${168 * M_PI / 180}"
-				 k_position="${100}"
-				 k_velocity="${2}"/>-->
       <parent link="arm_link_1"/>
       <child link="arm_link_2"/>
@@ -94,8 +82,4 @@
       <axis xyz="-1 0 0"/>
       <limit lower="${-180 * M_PI / 180}" upper="${180 * M_PI / 180}" effort="1000" velocity="${1.0 * 110 * M_PI / 180}"/>
-      <!--        <safety_controller soft_lower_limit="${-168 * M_PI / 180}"
-			 soft_upper_limit="${168 * M_PI / 180}"
-			 k_position="${100}"
-			 k_velocity="${2}"/>-->
       <parent link="arm_link_2"/>
       <child link="arm_link_3"/>
@@ -118,57 +102,4 @@
       <arm_link_3_collision_geom_marco/>
     </link>
-    <!--Needed for simulation-->
-    <transmission name="arm_joint_0_joint_transmssion">
-      <type>transmission_interface/SimpleTransmission</type>
-      <joint name="arm_joint_0">
-        <hardwareInterface>EffortJointInterface</hardwareInterface>
-      </joint>
-      <actuator name="arm_joint_0_motor">
-        <hardwareInterface>EffortJointInterface</hardwareInterface>
-        <mechanicalReduction>1</mechanicalReduction>
-      </actuator>
-    </transmission>
-    <transmission name="arm_joint_1_joint_transmssion">
-      <type>transmission_interface/SimpleTransmission</type>
-      <joint name="arm_joint_1">
-        <hardwareInterface>EffortJointInterface</hardwareInterface>
-      </joint>
-      <actuator name="arm_joint_1_motor">
-        <hardwareInterface>EffortJointInterface</hardwareInterface>
-        <mechanicalReduction>1</mechanicalReduction>
-      </actuator>
-    </transmission>
-    <transmission name="arm_joint_2_joint_transmssion">
-      <type>transmission_interface/SimpleTransmission</type>
-      <joint name="arm_joint_2">
-        <hardwareInterface>EffortJointInterface</hardwareInterface>
-      </joint>
-      <actuator name="arm_joint_2_motor">
-        <hardwareInterface>EffortJointInterface</hardwareInterface>
-        <mechanicalReduction>1</mechanicalReduction>
-      </actuator>
-    </transmission>
-    <transmission name="arm_joint_3_joint_transmssion">
-      <type>transmission_interface/SimpleTransmission</type>
-      <joint name="arm_joint_3">
-        <hardwareInterface>EffortJointInterface</hardwareInterface>
-      </joint>
-      <actuator name="arm_joint_3_motor">
-        <hardwareInterface>EffortJointInterface</hardwareInterface>
-        <mechanicalReduction>1</mechanicalReduction>
-      </actuator>
-    </transmission>
-    <gazebo reference="arm_link_0">
-      <material>Gazebo/Grey</material>
-    </gazebo>
-    <gazebo reference="arm_link_1">
-      <material>Gazebo/Grey</material>
-    </gazebo>
-    <gazebo reference="arm_link_2">
-      <material>Gazebo/Grey</material>
-    </gazebo>
-    <gazebo reference="arm_link_3">
-      <material>Gazebo/Grey</material>
-    </gazebo>
   </xacro:macro>
 </robot>
