Commit message: libtaurob and the description package ported

File: taurob_tracker_description/urdf/tracker_chassis.urdf.xacro (robot description, xacro)
@@ -1,68 +1,364 @@
 <?xml version="1.0"?>
-<robot xmlns:xacro="http://www.ros.org/wiki/xacro" name="taurob_tracker">
-  <xacro:include filename="$(find hector_xacro_tools)/urdf/inertia_tensors.urdf.xacro"/>
-  <xacro:property name="base_size_x" value="${0.365*2}"/>
-  <xacro:property name="base_size_y" value="0.24"/>
-  <xacro:property name="base_size_z" value="0.312 "/>
-  <xacro:property name="base_offset_x" value="-0.122"/>
-  <xacro:property name="base_offset_z" value="-0.05"/>
+<robot name="taurob_tracker" xmlns:xacro="http://www.ros.org/wiki/xacro" >
+  <xacro:include filename="$(find hector_xacro_tools)/urdf/inertia_tensors.urdf.xacro" />
+  <!--xacro:include filename="$(find taurob_tracker_description)/urdf/tracker_chassis.gazebo.xacro.xml" /-->
   <xacro:macro name="tracker_chassis_macro">
+    <xacro:property name="tracker_base_size_x" value="1.0" />
+    <xacro:property name="tracker_base_size_y" value="0.5" />
+    <xacro:property name="tracker_base_size_z" value="0.2 " />
+    <xacro:property name="tracker_base_offset_x" value="-0.122" />
+    <xacro:property name="tracker_base_offset_z" value="-0.08" />
+    <xacro:property name="flipper_offset_x" value="-0.051" />
+    <xacro:property name="flipper_upper_shortening_x" value="0.05" />
+    <!-- width overall is 0.58 ->  (0.58 - 0.0925)/2 = 0.24375 -->
+    <xacro:property name="track_offset_y" value="0.24375" />
+    <!--Below pending clarification-->
+    <xacro:property name="track_offset_z" value="-0.09" />
+    <xacro:property name="track_wheel_radius" value="0.13" />
+    <xacro:property name="track_width" value="0.0925" />
+    <!--no gazebo tags
+    <xacro:tracker_chassis_gazebo_force_based_move_macro />
+    <xacro:tracker_flipper_move_gazebo_macro />
+    -->
     <link name="base_link"/>
     <joint name="chassis_joint" type="fixed">
-      <origin xyz="${-base_offset_x} 0 0.18" rpy="0 0 0"/>
+      <origin xyz="${-tracker_base_offset_x} 0 0.193" rpy="0 0 0"/>
       <parent link="base_link"/>
       <child link="chassis_link"/>
     </joint>
-    <link name="flipper_link">
-      <origin xyz="0 0 0" rpy="0 0 0"/>
-      <collision>
-        <origin xyz="0.5 -0.23 ${base_offset_z}" rpy="0 0 0"/>
-        <geometry>
-          <box size="1.05 0.14 0.35"/>
-        </geometry>
-      </collision>
-      <collision>
-        <origin xyz="0.5 0.23 ${base_offset_z}" rpy="0 0 0"/>
-        <geometry>
-          <box size="1.05 0.14 0.35"/>
+    <link name="flipper_link_0">
+      <xacro:inertial_cuboid_with_pose mass="2.0" x_length="${tracker_base_size_x*0.25}" y_length="${track_width*2}" z_length="0.17651" >
+        <origin xyz="0.0 0.0 0.0" rpy="0 0 0" />
+      </xacro:inertial_cuboid_with_pose>
+      <origin xyz="0 0 0" rpy="0 0 0" />
+      <visual>
+        <origin xyz="${tracker_base_size_x-2*track_wheel_radius-flipper_upper_shortening_x} -${track_offset_y} 0.0" rpy="${pi/2} 0 0"/>
+        <geometry>
+          <cylinder length="${track_width}" radius="${track_wheel_radius}"/>
+        </geometry>
+        <material name="black">
+          <color rgba="0 0 0 1"/>
+        </material>
+      </visual>
+      <visual>
+        <origin xyz="0 -${track_offset_y} 0.0" rpy="${pi/2} 0 0"/>
+        <geometry>
+          <cylinder length="${track_width}" radius="${track_wheel_radius}"/>
+        </geometry>
+         <material name="black">
+          <color rgba="0 0 0 1"/>
+        </material>
+      </visual>
+      <visual>
+        <origin xyz="${tracker_base_size_x*0.5-track_wheel_radius-flipper_upper_shortening_x*0.5} -${track_offset_y} 0.0" rpy="0 0 0"/>
+        <geometry>
+          <box size="${tracker_base_size_x-2*track_wheel_radius-flipper_upper_shortening_x} ${track_width} ${track_wheel_radius*2}"/>
+        </geometry>
+        <material name="black">
+          <color rgba="0 0 0 1"/>
+        </material>
+      </visual>
+      <visual>
+        <origin xyz="${tracker_base_size_x-2*track_wheel_radius-flipper_upper_shortening_x} ${track_offset_y} 0.0" rpy="${pi/2} 0 0"/>
+        <geometry>
+          <cylinder length="${track_width}" radius="${track_wheel_radius}"/>
+        </geometry>
+        <material name="black">
+          <color rgba="0 0 0 1"/>
+        </material>
+      </visual>
+      <visual>
+        <origin xyz="0 ${track_offset_y} 0.0" rpy="${pi/2} 0 0"/>
+        <geometry>
+          <cylinder length="${track_width}" radius="${track_wheel_radius}"/>
+        </geometry>
+        <material name="black">
+          <color rgba="0 0 0 1"/>
+        </material>
+      </visual>
+      <visual>
+        <origin xyz="${tracker_base_size_x*0.5-track_wheel_radius-flipper_upper_shortening_x*0.5} ${track_offset_y} 0.0" rpy="0 0 0"/>
+        <geometry>
+          <box size="${tracker_base_size_x-2*track_wheel_radius-flipper_upper_shortening_x} ${track_width} ${track_wheel_radius*2}"/>
+        </geometry>
+        <material name="black">
+          <color rgba="0 0 0 1"/>
+        </material>
+      </visual>
+      <collision>
+        <origin xyz="${tracker_base_size_x-2*track_wheel_radius} -${track_offset_y} 0.0" rpy="${pi/2} 0 0"/>
+        <geometry>
+          <cylinder length="${track_width}" radius="${track_wheel_radius}"/>
+        </geometry>
+      </collision>
+      <collision>
+        <origin xyz="0 -${track_offset_y} 0.0" rpy="${pi/2} 0 0"/>
+        <geometry>
+          <cylinder length="${track_width}" radius="${track_wheel_radius}"/>
+        </geometry>
+      </collision>
+      <collision>
+        <origin xyz="${tracker_base_size_x*0.5-track_wheel_radius} -${track_offset_y} 0.0" rpy="0 0 0"/>
+        <geometry>
+          <box size="${tracker_base_size_x-2*track_wheel_radius} ${track_width} ${track_wheel_radius*2}"/>
+        </geometry>
+      </collision>
+      <collision>
+        <origin xyz="${tracker_base_size_x-2*track_wheel_radius} ${track_offset_y} 0.0" rpy="${pi/2} 0 0"/>
+        <geometry>
+          <cylinder length="${track_width}" radius="${track_wheel_radius}"/>
+        </geometry>
+      </collision>
+      <collision>
+        <origin xyz="0 ${track_offset_y} 0.0" rpy="${pi/2} 0 0"/>
+        <geometry>
+          <cylinder length="${track_width}" radius="${track_wheel_radius}"/>
+        </geometry>
+      </collision>
+      <collision>
+        <origin xyz="${tracker_base_size_x*0.5-track_wheel_radius} ${track_offset_y} 0.0" rpy="0 0 0"/>
+        <geometry>
+          <box size="${tracker_base_size_x-2*track_wheel_radius} ${track_width} ${track_wheel_radius*2}"/>
         </geometry>
       </collision>
     </link>
-    <joint name="flipper_front" type="revolute">
-      <origin xyz="${base_offset_x-0.5} 0 0" rpy="0 0 0"/>
-      <axis xyz="0 -1 0"/>
-      <limit lower="${-30 * M_PI / 180}" upper="${50 * M_PI / 180}" effort="204" velocity="${1.0 * 110 * M_PI / 180}"/>
-      <safety_controller soft_lower_limit="${-25 * M_PI / 180}" soft_upper_limit="${45 * M_PI / 180}" k_position="${100}" k_velocity="${2}"/>
+    <joint name="flipper_joint_0" type="revolute">
+      <origin xyz="${tracker_base_offset_x-(tracker_base_size_x*0.5-track_wheel_radius)} 0 ${track_offset_z}" rpy="0 0 0" />
+      <axis xyz="0 1 0"/>
+      <mimic joint="flipper_joint_1" multiplier="0.46"/>
+      <limit lower="${-170 * pi / 180}" upper="${180 * pi / 180}"
+             effort="10000" velocity="${10.0 * 360 * pi / 180}" />
+<!--      <safety_controller soft_lower_limit="${-25 * pi / 180}"
+                         soft_upper_limit="${45 * pi / 180}"
+                         k_position="${100}"
+                         k_velocity="${2}"/>-->
       <parent link="chassis_link"/>
-      <child link="flipper_link"/>
+      <child link="flipper_link_0"/>
     </joint>
+    <!--Needed for simulation-->
+    <transmission name="flipper_joint_0_joint_transmssion">
+      <type>transmission_interface/SimpleTransmission</type>
+      <joint name="flipper_joint_0">
+        <hardwareInterface>EffortJointInterface</hardwareInterface>
+      </joint>
+      <actuator name="flipper_joint_0_motor">
+        <hardwareInterface>EffortJointInterface</hardwareInterface>
+        <mechanicalReduction>1</mechanicalReduction>
+      </actuator>
+    </transmission>
+    <link name="flipper_link_1">
+      <xacro:inertial_cuboid_with_pose mass="1.0" x_length="${tracker_base_size_x*0.5}" y_length="${track_width*2}" z_length="0.17651" >
+        <origin xyz="${tracker_base_size_x*0.5-track_wheel_radius*2} 0.0 0.0" rpy="0 0 0" />
+      </xacro:inertial_cuboid_with_pose>
+      <origin xyz="0 0 0" rpy="0 0 0" />
+      <visual>
+        <origin xyz="${tracker_base_size_x*0.5-track_wheel_radius+flipper_offset_x} -${track_offset_y} 0.0" rpy="${pi/2} 0 0"/>
+        <geometry>
+          <cylinder length="${track_width}" radius="${track_wheel_radius}"/>
+        </geometry>
+        <material name="black">
+          <color rgba="0 0 0 1"/>
+        </material>
+      </visual>
+      <visual>
+        <origin xyz="0 -${track_offset_y} 0.0" rpy="${pi/2} 0 0"/>
+        <geometry>
+          <cylinder length="${track_width}" radius="${track_wheel_radius}"/>
+        </geometry>
+        <material name="black">
+          <color rgba="0 0 0 1"/>
+        </material>
+      </visual>
+      <visual>
+        <origin xyz="${(tracker_base_size_x*0.5-track_wheel_radius+flipper_offset_x)*0.5} -${track_offset_y} 0.0" rpy="0 0 0"/>
+        <geometry>
+          <box size="${tracker_base_size_x*0.5-track_wheel_radius+flipper_offset_x} ${track_width} ${track_wheel_radius*2}"/>
+        </geometry>
+        <material name="black">
+          <color rgba="0 0 0 1"/>
+        </material>
+      </visual>
+      <visual>
+        <origin xyz="${tracker_base_size_x*0.5-track_wheel_radius+flipper_offset_x} ${track_offset_y} 0.0" rpy="${pi/2} 0 0"/>
+        <geometry>
+          <cylinder length="${track_width}" radius="${track_wheel_radius}"/>
+        </geometry>
+        <material name="black">
+          <color rgba="0 0 0 1"/>
+        </material>
+      </visual>
+      <visual>
+        <origin xyz="0 ${track_offset_y} 0.0" rpy="${pi/2} 0 0"/>
+        <geometry>
+          <cylinder length="${track_width}" radius="${track_wheel_radius}"/>
+        </geometry>
+        <material name="black">
+          <color rgba="0 0 0 1"/>
+        </material>
+      </visual>
+      <visual>
+        <origin xyz="${(tracker_base_size_x*0.5-track_wheel_radius+flipper_offset_x)*0.5} ${track_offset_y} 0.0" rpy="0 0 0"/>
+        <geometry>
+          <box size="${tracker_base_size_x*0.5-track_wheel_radius+flipper_offset_x} ${track_width} ${track_wheel_radius*2}"/>
+        </geometry>
+        <material name="black">
+          <color rgba="0 0 0 1"/>
+        </material>
+      </visual>
+      <collision>
+        <origin xyz="${tracker_base_size_x*0.5-track_wheel_radius+flipper_offset_x} -${track_offset_y} 0.0" rpy="${pi/2} 0 0"/>
+        <geometry>
+          <cylinder length="${track_width}" radius="${track_wheel_radius}"/>
+        </geometry>
+      </collision>
+      <collision>
+        <origin xyz="0 -${track_offset_y} 0.0" rpy="${pi/2} 0 0"/>
+        <geometry>
+          <cylinder length="${track_width}" radius="${track_wheel_radius}"/>
+        </geometry>
+      </collision>
+      <collision>
+        <origin xyz="${(tracker_base_size_x*0.5-track_wheel_radius+flipper_offset_x)*0.5} -${track_offset_y} 0.0" rpy="0 0 0"/>
+        <geometry>
+          <box size="${tracker_base_size_x*0.5-track_wheel_radius+flipper_offset_x} ${track_width} ${track_wheel_radius*2}"/>
+        </geometry>
+      </collision>
+      <collision>
+        <origin xyz="${tracker_base_size_x*0.5-track_wheel_radius+flipper_offset_x} ${track_offset_y} 0.0" rpy="${pi/2} 0 0"/>
+        <geometry>
+          <cylinder length="${track_width}" radius="${track_wheel_radius}"/>
+        </geometry>
+      </collision>
+      <collision>
+        <origin xyz="0 ${track_offset_y} 0.0" rpy="${pi/2} 0 0"/>
+        <geometry>
+          <cylinder length="${track_width}" radius="${track_wheel_radius}"/>
+        </geometry>
+      </collision>
+      <collision>
+        <origin xyz="${(tracker_base_size_x*0.5-track_wheel_radius+flipper_offset_x)*0.5} ${track_offset_y} 0.0" rpy="0 0 0"/>
+        <geometry>
+          <box size="${tracker_base_size_x*0.5-track_wheel_radius+flipper_offset_x} ${track_width} ${track_wheel_radius*2}"/>
+        </geometry>
+      </collision>
+    </link>
+    <joint name="flipper_joint_1" type="revolute">
+      <origin xyz="${tracker_base_offset_x-flipper_offset_x} 0 ${track_offset_z}" rpy="0 0 0" />
+      <axis xyz="0 1 0"/>
+      <limit lower="${-50 * pi / 180}" upper="${30 * pi / 180}"
+             effort="10000" velocity="${1.0 * 30 * pi / 180}" />
+<!--      <safety_controller soft_lower_limit="${-25 * pi / 180}"
+                         soft_upper_limit="${45 * pi / 180}"
+                         k_position="${100}"
+                         k_velocity="${2}"/>-->
+      <parent link="chassis_link"/>
+      <child link="flipper_link_1"/>
+    </joint>
+    <!--Needed for simulation-->
+    <transmission name="flipper_joint_1_joint_transmssion">
+      <type>transmission_interface/SimpleTransmission</type>
+      <joint name="flipper_joint_1">
+        <hardwareInterface>EffortJointInterface</hardwareInterface>
+      </joint>
+      <actuator name="flipper_joint_1_motor">
+        <hardwareInterface>EffortJointInterface</hardwareInterface>
+        <mechanicalReduction>1</mechanicalReduction>
+      </actuator>
+    </transmission>
     <link name="chassis_link">
-      <xacro:inertial_cuboid_with_pose mass="20" x_length="${base_size_x}" y_length="${base_size_y}" z_length="${base_size_z}">
-        <origin xyz="0.0 0.0 ${0.312*0.5}" rpy="0 0 0"/>
+      <xacro:inertial_cuboid_with_pose mass="30" x_length="${tracker_base_size_x*0.66}" y_length="${tracker_base_size_y}" z_length="${tracker_base_size_z}" >
+        <origin xyz="${-tracker_base_size_x*0.25} 0.0 -0.05" rpy="0 0 0" />
       </xacro:inertial_cuboid_with_pose>
-      <visual>
-        <origin xyz="0.0 0.0 0.0" rpy="0 0 0"/>
-        <geometry>
-          <mesh filename="package://taurob_tracker_description/meshes/tracker_chassis.dae"/>
-        </geometry>
-      </visual>
-      <collision>
-        <origin xyz="${base_offset_x-0.11} 0.0 ${base_offset_z}" rpy="0 0 0"/>
-        <geometry>
-          <box size="0.74 0.5 0.2"/>
-        </geometry>
-      </collision>
-      <collision>
-        <origin xyz="${base_offset_x} -0.23 ${base_offset_z}" rpy="0 0 0"/>
-        <geometry>
-          <box size="1.0 0.13 0.35"/>
-        </geometry>
-      </collision>
-      <collision>
-        <origin xyz="${base_offset_x} 0.23 ${base_offset_z}" rpy="0 0 0"/>
-        <geometry>
-          <box size="1.0 0.13 0.35"/>
-        </geometry>
-      </collision>
+      <!--Primitives with materials need to be used before .dae, otherwise material does not get applied-->
+      <visual>
+        <origin xyz="${tracker_base_offset_x - flipper_offset_x - (tracker_base_size_x*0.5-track_wheel_radius-flipper_offset_x)*0.5} -${track_offset_y} ${track_offset_z}" rpy="0 0 0"/>
+        <geometry>
+          <mesh filename="package://taurob_tracker_description/meshes/tracker_chassis_sides.dae"/>
+        </geometry>
+        <material name="black">
+          <color rgba="0 0 0 1"/>
+        </material>
+      </visual>
+      <visual>
+        <origin xyz="${tracker_base_offset_x - flipper_offset_x - (tracker_base_size_x*0.5-track_wheel_radius-flipper_offset_x)*0.5} ${track_offset_y} ${track_offset_z}" rpy="0 0 0"/>
+        <geometry>
+          <mesh filename="package://taurob_tracker_description/meshes/tracker_chassis_sides.dae"/>
+        </geometry>
+        <material name="black">
+          <color rgba="0 0 0 1"/>
+        </material>
+      </visual>
+      <visual>
+        <origin xyz="0.0 0.0 0.0" rpy="0 0 0" />
+        <geometry>
+          <mesh filename="package://taurob_tracker_description/meshes/tracker_chassis_no_tracks.dae"/>
+        </geometry>
+      </visual>
+      <!--Left/right track box geoms-->
+      <collision>
+        <origin xyz="${tracker_base_offset_x - flipper_offset_x - (tracker_base_size_x*0.5-track_wheel_radius-flipper_offset_x)*0.5} -${track_offset_y} ${track_offset_z}" rpy="0 0 0"/>
+        <geometry>
+          <box size="${tracker_base_size_x*0.5-track_wheel_radius-flipper_offset_x} ${track_width} ${track_wheel_radius*2}"/>
+        </geometry>
+      </collision>
+      <collision>
+        <origin xyz="${tracker_base_offset_x - flipper_offset_x - (tracker_base_size_x*0.5-track_wheel_radius-flipper_offset_x)*0.5}  ${track_offset_y} ${track_offset_z}" rpy="0 0 0"/>
+        <geometry>
+          <box size="${tracker_base_size_x*0.5-track_wheel_radius-flipper_offset_x} ${track_width} ${track_wheel_radius*2}"/>
+        </geometry>
+      </collision>
+	  <!--Left/right back track cylinder geoms-->
+      <collision>
+        <origin xyz="${tracker_base_offset_x-(tracker_base_size_x*0.5-track_wheel_radius)} -${track_offset_y} ${track_offset_z}" rpy="${pi/2} 0 0"/>
+        <geometry>
+          <cylinder length="${track_width}" radius="${track_wheel_radius}"/>
+        </geometry>
+        <material name="red">
+          <color rgba="1 0 0 1"/>
+        </material>
+      </collision>
+      <collision>
+        <origin xyz="${tracker_base_offset_x-(tracker_base_size_x*0.5-track_wheel_radius)} ${track_offset_y} ${track_offset_z}" rpy="${pi/2} 0 0"/>
+        <geometry>
+          <cylinder length="${track_width}" radius="${track_wheel_radius}"/>
+        </geometry>
+      </collision>
+      <!--Chassis middle-->
+      <collision>
+        <origin xyz="${tracker_base_offset_x-0.13} 0.0 ${tracker_base_offset_z+0.005}" rpy="0 0 0"/>
+        <geometry>
+          <box size="0.7 0.5 0.15"/>
+        </geometry>
+      </collision>
+      <!--Left track cylinder (front/back) geoms-->
+      <!--
+      <collision>
+        <origin xyz="${tracker_base_offset_x + tracker_base_size_x*0.5 - track_wheel_radius} ${track_offset_y} ${tracker_base_offset_z}" rpy="${pi*0.5} 0 0"/>
+        <geometry>
+          <cylinder radius="${track_wheel_radius}" length="${track_width}" />
+        </geometry>
+      </collision>
+      <collision>
+        <origin xyz="${tracker_base_offset_x -tracker_base_size_x*0.5 + track_wheel_radius} ${track_offset_y} ${tracker_base_offset_z}" rpy="${pi*0.5} 0 0"/>
+        <geometry>
+          <cylinder radius="${track_wheel_radius}" length="${track_width}" />
+        </geometry>
+      </collision>
+      -->
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