Commit message: Port libtaurob_claw and add TrackerClawHardware ros2_control interface
Move the claw communication library (Claw, Claw_frames) from the ROS 1
master branch into libtaurob, converting the ODR-used static const
members to static constexpr and declaring the new boost-regex
dependency.

TrackerClawHardware exposes claw_rotation and claw_grip position
joints plus a claw force sensor state interface, is watchdog-gated
like all tracker actuation (holds current pose when unfed), and is
exported as a pluginlib SystemInterface. Add the claw ros2_control
block to the URDF, a claw_controller to the bringup config and its
spawner to the launch file.

Co-authored-by: tstoyanov <tstoyanov@users.noreply.github.com>

File: taurob_tracker_description/urdf/tracker_ros2_control.urdf.xacro (robot description, xacro)
@@ -40,4 +40,24 @@
         <state_interface name="position"/>
       </joint>
+    </ros2_control>
+    <!-- Claw: rotation and grip position joints plus grip force sensor -->
+    <ros2_control name="tracker_claw" type="system">
+      <hardware>
+        <plugin>taurob_tracker_hardware/TrackerClawHardware</plugin>
+        <param name="claw_ip">10.0.0.2</param>
+        <param name="claw_port">10003</param>
+        <param name="watchdog_enabled">${watchdog_enabled}</param>
+      </hardware>
+      <joint name="claw_rotation">
+        <command_interface name="position"/>
+        <state_interface name="position"/>
+      </joint>
+      <joint name="claw_grip">
+        <command_interface name="position"/>
+        <state_interface name="position"/>
+      </joint>
+      <sensor name="claw_force_sensor">
+        <state_interface name="force"/>
+      </sensor>
     </ros2_control>
     <!-- Arm: per-joint ECU addresses follow the ROS 1 tracker.yaml calibration

Commit message: URDF: add track joints for diff drive control
The kinematic model has no discrete wheel joints (tracked base), so add
abstract continuous track_left/track_right joints parented to base_link
solely for the ros2_control base system; TrackerBaseSystem correctly
rejected the URDF without them.

Co-authored-by: tstoyanov <tstoyanov@users.noreply.github.com>

File: taurob_tracker_description/urdf/tracker_ros2_control.urdf.xacro (robot description, xacro)
@@ -4,4 +4,21 @@
                                                    gear_ratio:='76.0' wheel_diameter:='0.303'
                                                    track_width:='0.55' watchdog_enabled:='true'">
+    <!-- Abstract wheel joints representing the two tracks for diff_drive_controller.
+         The tracks themselves have no discrete wheel joints in the kinematic model,
+         so these exist solely for ros2_control. -->
+    <link name="track_left_link"/>
+    <link name="track_right_link"/>
+    <joint name="track_left" type="continuous">
+      <parent link="base_link"/>
+      <child link="track_left_link"/>
+      <origin xyz="0 ${track_width / 2} 0" rpy="0 ${M_PI / 2} 0"/>
+      <axis xyz="0 0 1"/>
+    </joint>
+    <joint name="track_right" type="continuous">
+      <parent link="base_link"/>
+      <child link="track_right_link"/>
+      <origin xyz="0 -${track_width / 2} 0" rpy="0 ${M_PI / 2} 0"/>
+      <axis xyz="0 0 1"/>
+    </joint>
     <!-- Base drivetrain: diff drive on the two tracks -->
     <ros2_control name="tracker_base" type="system">

Commit message: URDF: cast track_width to float in xacro origin expressions
Co-authored-by: tstoyanov <tstoyanov@users.noreply.github.com>

File: taurob_tracker_description/urdf/tracker_ros2_control.urdf.xacro (robot description, xacro)
@@ -12,5 +12,5 @@
       <parent link="base_link"/>
       <child link="track_left_link"/>
-      <origin xyz="0 ${track_width / 2} 0" rpy="0 ${M_PI / 2} 0"/>
+      <origin xyz="0 ${float(track_width) / 2} 0" rpy="0 ${M_PI / 2} 0"/>
       <axis xyz="0 0 1"/>
     </joint>
@@ -18,5 +18,5 @@
       <parent link="base_link"/>
       <child link="track_right_link"/>
-      <origin xyz="0 -${track_width / 2} 0" rpy="0 ${M_PI / 2} 0"/>
+      <origin xyz="0 -${float(track_width) / 2} 0" rpy="0 ${M_PI / 2} 0"/>
       <axis xyz="0 0 1"/>
     </joint>

Commit message: URDF: add abstract flipper and claw joints for ros2_control
Co-authored-by: tstoyanov <tstoyanov@users.noreply.github.com>

File: taurob_tracker_description/urdf/tracker_ros2_control.urdf.xacro (robot description, xacro)
@@ -20,4 +20,25 @@
       <origin xyz="0 -${float(track_width) / 2} 0" rpy="0 ${M_PI / 2} 0"/>
       <axis xyz="0 0 1"/>
+    </joint>
+    <!-- Abstract joints for the flipper and claw (the kinematic chassis model
+         uses flipper_joint_0/1; these exist solely for ros2_control). -->
+    <link name="flipper_front_link"/>
+    <joint name="flipper_front" type="continuous">
+      <parent link="base_link"/>
+      <child link="flipper_front_link"/>
+      <origin xyz="${float(flipper_offset_x)} 0 ${float(flipper_offset_z)}"/>
+      <axis xyz="0 1 0"/>
+    </joint>
+    <link name="claw_rotation_link"/>
+    <link name="claw_grip_link"/>
+    <joint name="claw_rotation" type="continuous">
+      <parent link="arm_link_3"/>
+      <child link="claw_rotation_link"/>
+      <axis xyz="0 0 1"/>
+    </joint>
+    <joint name="claw_grip" type="continuous">
+      <parent link="claw_rotation_link"/>
+      <child link="claw_grip_link"/>
+      <axis xyz="0 1 0"/>
     </joint>
     <!-- Base drivetrain: diff drive on the two tracks -->
